Commit message: Teleop Final

File: capulus/urdf/capulus.urdf (robot description, URDF)
Before this commit: robot capulus, 3 links, 2 joints
Links:
- added link imu; visual box size=0.01 0.01 0.01
Joints:
- added joint imu_joint: type fixed, parent base_link, child imu, origin xyz=0 0 0.05 rpy=0 0 0
- joint base_to_wheel1: origin xyz=0 0 0 rpy=0 0 0 -> xyz=0 0 0 rpy=0 0 1.57079632679
- joint base_to_wheel2: origin xyz=0 0 0 rpy=0 0 0 -> xyz=0 0 0 rpy=0 0 1.57079632679
